File: PCB/ESC_Device_Hub_v0/ESC_Device_Hub_v0.kicad_sch (KiCad schematic)
At the start: 0 parts

Commit message: 部品配置９割終わった
Parts:
- added C1, C2, C3, C5: 0.1uF, Capacitor_SMD:C_0603_1608Metric_Pad1.08x0.95mm_HandSolder, symbol Device:C_Small
- added C10, C8: 2.2uF, Capacitor_SMD:C_0603_1608Metric_Pad1.08x0.95mm_HandSolder, symbol Device:C_Small
- added C11: 0.33uF, Capacitor_SMD:C_0603_1608Metric_Pad1.08x0.95mm_HandSolder, symbol Device:C_Small
- added C12, C13, C14, C15, C16, C17, C18, C19, C21, C23, C25, C27, C28, C29, C4, C7: 0.1uF, Capacitor_SMD:C_0402_1005Metric_Pad0.74x0.62mm_HandSolder, symbol Device:C_Small
- added C20: 4.7uF, Capacitor_SMD:C_0402_1005Metric_Pad0.74x0.62mm_HandSolder, symbol Device:C_Small
- added C22, C24, C32: 1uF, Capacitor_SMD:C_0402_1005Metric_Pad0.74x0.62mm_HandSolder, symbol Device:C_Small
- added C26: 2.2uF, Capacitor_SMD:C_0402_1005Metric_Pad0.74x0.62mm_HandSolder, symbol Device:C_Small
- added C30, C31: 8pF, Capacitor_SMD:C_0402_1005Metric_Pad0.74x0.62mm_HandSolder, symbol Device:C_Small
- added C6: 0.01uF, Capacitor_SMD:C_0603_1608Metric_Pad1.08x0.95mm_HandSolder, symbol Device:C
- added C9: 47uF, Capacitor_SMD:C_0603_1608Metric_Pad1.08x0.95mm_HandSolder, symbol Device:C_Small
- added D1, D12, D2, D7, D8, D9: W, LED_SMD:LED_0603_1608Metric_Pad1.05x0.95mm_HandSolder, symbol Device:LED
- added D10, D11, D16, D17, D22, D23, D25, D26: LED, LED_SMD:LED_0603_1608Metric_Pad1.05x0.95mm_HandSolder, symbol Device:LED
- added D13: SS2040FL, My_Library:SS2040FL, symbol Device:D_Filled
- added D3, D4: R, LED_SMD:LED_0603_1608Metric_Pad1.05x0.95mm_HandSolder, symbol Device:LED
- added D5: B, LED_SMD:LED_0603_1608Metric_Pad1.05x0.95mm_HandSolder, symbol Device:LED
- added D6: G, LED_SMD:LED_0603_1608Metric_Pad1.05x0.95mm_HandSolder, symbol Device:LED
- added FB1: 600Ω/500mA, Inductor_SMD:L_0603_1608Metric_Pad1.05x0.95mm_HandSolder, symbol Device:FerriteBead
- added J1, J2: Conn_01x04, Connector_JST:JST_XH_S4B-XH-A_1x04_P2.50mm_Horizontal, symbol Connector_Generic:Conn_01x04
- added J10, J7, J8, J9: Conn_01x06, Connector_JST:JST_XH_B6B-XH-A_1x06_P2.50mm_Vertical, symbol Connector_Generic:Conn_01x06
- added J11, J12, J13, J14, J15, J16, J17, J18: Conn_01x02, Connector_JST:JST_XH_B2B-XH-A_1x02_P2.50mm_Vertical, symbol Connector_Generic:Conn_01x02
- added J19: Conn_01x05, Connector_PinSocket_2.54mm:PinSocket_1x05_P2.54mm_Vertical, symbol Connector_Generic:Conn_01x05
- added J20, J21: Conn_01x01, 0Ikedalibrary:5x5, symbol Connector_Generic:Conn_01x01
- added J22: Conn_01x02, Connector_JST:JST_XH_S2B-XH-A_1x02_P2.50mm_Horizontal, symbol Connector_Generic:Conn_01x02
- added J3, J4, J5, J6: Conn_01x04, Connector_JST:JST_XH_B4B-XH-A_1x04_P2.50mm_Vertical, symbol Connector_Generic:Conn_01x04
- added JP1, JP2: Jumper_2_Bridged, Connector_PinHeader_2.54mm:PinHeader_1x02_P2.54mm_Vertical, symbol Jumper:Jumper_2_Bridged
- added L1: 22uH, My_Library:SRP4020TA-220M, symbol Device:L
- added R1, R2, R4: 120, Resistor_SMD:R_0603_1608Metric_Pad0.98x0.95mm_HandSolder, symbol Device:R
- added R10, R11, R12, R13, R14, R15, R16, R17, R19, R20, R21, R22, R23, R56, R8: 1k, Resistor_SMD:R_0603_1608Metric_Pad0.98x0.95mm_HandSolder, symbol Device:R_Small
- added R18: 1k, Resistor_SMD:R_0402_1005Metric_Pad0.72x0.64mm_HandSolder, symbol Device:R_Small
- added R3: 10k, Resistor_SMD:R_0402_1005Metric_Pad0.72x0.64mm_HandSolder, symbol Device:R_Small
- added R43, R44, R51, R52, R59, R60, R65, R66: 22k, Resistor_SMD:R_0603_1608Metric_Pad0.98x0.95mm_HandSolder, symbol Device:R
- added R46, R47, R5, R54, R55, R62, R63, R67, R68: 1k, Resistor_SMD:R_0603_1608Metric_Pad0.98x0.95mm_HandSolder, symbol Device:R
- added R6: 3.9k, Resistor_SMD:R_0603_1608Metric_Pad0.98x0.95mm_HandSolder, symbol Device:R_Small
- added R7: 1.2k, Resistor_SMD:R_0603_1608Metric_Pad0.98x0.95mm_HandSolder, symbol Device:R_Small
- added R77, R78: 4.7k, Resistor_SMD:R_0402_1005Metric_Pad0.72x0.64mm_HandSolder, symbol Device:R
- added R9: 10k, Resistor_SMD:R_0603_1608Metric_Pad0.98x0.95mm_HandSolder, symbol Device:R_Small
- added SW1, SW2: SW_Push, 0Ikedalibrary:switch_TVAF06-A020B-R, symbol Switch:SW_Push
- added SW3: SW_Coded_SH-7050, My_Library:ERD116RFZ, symbol Switch:SW_Coded_SH-7050
- added SW4: SW_DIP_x02, My_Library:KHS22E, symbol Switch:SW_DIP_x02
- added U1: ISO1042BQDWVRQ1, Package_SO:SOIC-8_7.5x5.85mm_P1.27mm, symbol My_Library:ISO1042B
- added U17: ~, My_Library:ECS-TXO-2520-33-500-AN-TR, symbol My_Library:ECS-TXO-2520-33-500-AN-TR
- added U18: USB_Type-C, 0Ikedalibrary:USB_C_Receptacle_Nelton_5077CR-16-SMC2-BK-TR, symbol My_Library:USB_Type-C
- added U2: MCP2562FD-H/MF, Package_DFN_QFN:DFN-8-1EP_3x3mm_P0.65mm_EP1.6x2.56mm, symbol My_Library:MCP2562FD-H/MF
- added U3: IS25LP064D-JLLE, Package_SON:WSON-8-1EP_8x6mm_P1.27mm_EP3.4x4.3mm, symbol My_Library:IS25LP064D
- added U4: STM32H563RGVx, Package_DFN_QFN:QFN-68-1EP_8x8mm_P0.4mm_EP6.4x6.4mm, symbol MCU_ST_STM32H5:STM32H563RGVx
- added U5: NJW1933F1-AT, Package_TO_SOT_SMD:SOT-23-6_Handsoldering, symbol My_Library:NJW1933F1
- added U6: TLP293, Package_SO:SOIC-4_4.55x2.6mm_P1.27mm, symbol Isolator:TLP293
- added U7: NJM2884U1-33, Package_TO_SOT_SMD:SOT-89-5, symbol My_Library:NJM2884U1-33
- added U8, U9: XC8114AA01PR-G, Package_TO_SOT_SMD:SOT-89-5, symbol My_Library:XC8114AA01PR-G
- added Y1: FC2012SN 32.768K-70NNA0KC0, My_Library:FC2012SN 32.768K-70NNA0KC0, symbol My_Library:FC2012SN
Connections:
- new net: R18.2, U7.1 (CONT)
- new net: D26.2 (A), R68.1
- new net: D7.2 (A), R15.2
- new net: D22.2 (A), R62.1
- new net: R6.1, R7.1, U5.3 (FB)
- new net: JP1.2 (B), R4.1
- new net: D10.2 (A), R46.1
- new net: C25.1, C26.1, U4.31 (VCAP)
- new net: D5.2 (A), R12.2
- new net: D25.2 (A), R67.1
- new net: D23.2 (A), R63.1
- new net: D17.2 (A), R55.1
- new net: R9.2, U6.1
- new net: D12.2 (A), R23.2
- new net: R78.1, U18.A5 (CC1)
- new net: D4.2 (A), R11.2
- new net: D11.2 (A), R47.1
- new net: D9.2 (A), R17.2
- new net: D6.2 (A), R13.2
- new net: D8.2 (A), R16.2
- new net: JP2.2 (B), R1.1
- new net: D13.1 (K), L1.1, U5.6 (Vout)
- new net: R5.1, SW3.C
- new net: R77.1, U18.B5 (CC2)
- new net: D3.2 (A), R10.2
- new net: D2.2 (A), R8.2
- new net: R56.1, U6.4
- new net: C27.1, C28.1, U4.66 (VCAP)
- new net: D1.2 (A), R14.2
- new net: D16.2 (A), R54.1
- new net: C12.1, FB1.2, U8.2 (EP), U8.4 (Vin)
- new net +3.3V: C10.1, C16.1, C17.1, C18.1, C19.1, C20.1, C21.1, C22.1, C23.1, C24.1, C29.1, C3.1, C32.1, C5.1, J10.5 (Pin_5), J19.5 (Pin_5), J7.5 (Pin_5), J8.5 (Pin_5), J9.5 (Pin_5), R17.1, R43.2, R44.2, R46.2, R47.2, R5.2, R51.2, R52.2, R54.2, R55.2, R56.2, R59.2, R60.2, R62.2, R63.2, R65.2, R66.2, R67.2, R68.2, SW2.1, SW4.1, SW4.2, U17.1 (Tri_state), U17.4 (VDD), U2.5 (Vio), U3.8 (Vcc), U4.1 (VBAT), U4.13 (VDDA), U4.19 (VDD), U4.33 (VDD), U4.51 (VDD), U4.68 (VDD), U7.5 (Vin)
- new net +5V: C11.1, C13.1, C15.1, C2.1, C4.1, R16.1, R18.1, U1.1 (VCC1), U2.3 (VDD), U7.4 (Vout), U8.5 (Vout), U9.5 (Vout)
- new net +5VA: C14.1, J1.3 (Pin_3), J2.3 (Pin_3), R15.1, U9.2 (EP), U9.4 (Vin)
- new net +5VP: C1.1, C9.1, J3.3 (Pin_3), J4.3 (Pin_3), J5.3 (Pin_3), J6.3 (Pin_3), L1.2, R7.2, R8.1, U1.8 (VCC2)
- new net BOOT0: R3.1, SW2.2, U4.62 (BOOT0)
- new net CAN_H: J1.4 (Pin_4), J2.4 (Pin_4), JP2.1 (A), U2.7 (CANH)
- new net CAN_L: J1.2 (Pin_2), J2.2 (Pin_2), R1.2, U2.6 (CANL)
- new net ENC1_A: J7.6 (Pin_6), U4.14 (PA0)
- new net ENC1_B: J7.4 (Pin_4), U4.15 (PA1)
- new net ENC2_A: J8.6 (Pin_6), U4.22 (PA6)
- new net ENC2_B: J8.4 (Pin_4), U4.23 (PA7)
- new net ENC3_A: J9.6 (Pin_6), U4.60 (PB6)
- new net ENC3_B: J9.4 (Pin_4), U4.61 (PB7)
- new net ENC4_A: J10.6 (Pin_6), U4.44 (PA8)
- new net ENC4_B: J10.4 (Pin_4), U4.45 (PA9)
- new net ESC_FDCAN_RXD: U1.3 (RXD), U4.34 (PB12)
- new net ESC_FDCAN_TXD: U1.2 (TXD), U4.35 (PB13)
- new net FDCAN_RXD: U2.4 (RXD), U4.63 (PB8)
- new net FDCAN_TXD: U2.1 (TXD), U4.64 (PB9)
- new net FLASH_IO0: U3.5 (SI(IO0)), U4.9 (PC1)
- new net FLASH_IO1: U3.2 (SO(IO1)), U4.10 (PC2)
- new net FLASH_IO2: U3.3 (WP(IO2)), U4.11 (PC3)
- new net FLASH_IO3: U3.7 (HOLD/RESET(IO3)), U4.8 (PC0)
- new net FLASH_SCK: U3.6 (SCK), U4.17 (PA3)
- new net FLASH_SS: U3.1 (CE#), U4.29 (PB10)
- new net GND: C10.2, C11.2, C12.2, C13.2, C14.2, C15.2, C16.2, C17.2, C18.2, C19.2, C2.2, C20.2, C21.2, C22.2, C23.2, C24.2, C25.2, C26.2, C27.2, C28.2, C29.2, C3.2, C30.2, C31.2, C32.2, C4.2, C5.2, C6.2, C7.2, D12.1 (K), D3.1 (K), D4.1 (K), D5.1 (K), D6.1 (K), D7.1 (K), D8.1 (K), D9.1 (K), J1.1 (Pin_1), J10.1 (Pin_1), J10.2 (Pin_2), J10.3 (Pin_3), J11.1 (Pin_1), J12.1 (Pin_1), J13.1 (Pin_1), J14.1 (Pin_1), J15.1 (Pin_1), J16.1 (Pin_1), J17.1 (Pin_1), J18.1 (Pin_1), J19.4 (Pin_4), J2.1 (Pin_1), J7.1 (Pin_1), J7.2 (Pin_2), J7.3 (Pin_3), J8.1 (Pin_1), J8.2 (Pin_2), J8.3 (Pin_3), J9.1 (Pin_1), J9.2 (Pin_2), J9.3 (Pin_3), R19.2, R20.2, R21.2, R22.2, R3.2, R77.2, R78.2, SW1.1, U1.4 (GND1), U17.2 (GND), U18.A1 (GND), U18.B1 (GND), U2.2 (VSS), U2.8 (STBY), U2.9 (EP), U3.4 (GND), U3.9 (GND), U4.12 (VSSA), U4.18 (VSS), U4.32 (VSS), U4.50 (VSS), U4.67 (VSS), U4.69 (VSS), U7.2 (GND), U8.1 (GND), U8.3 (EP), U9.1 (GND), U9.3 (EP)
- new net GNDD: C1.2, C8.2, C9.2, D1.1 (K), D13.2 (A), D2.1 (K), J21.1 (Pin_1), J3.1 (Pin_1), J4.1 (Pin_1), J5.1 (Pin_1), J6.1 (Pin_1), R6.2, U1.5 (GND2), U5.2 (GND), U6.2
- new net Isolation_FDCAN_H: J3.4 (Pin_4), J4.4 (Pin_4), J5.4 (Pin_4), J6.4 (Pin_4), JP1.1 (A), R2.1, U1.7 (CANH)
- new net Isolation_FDCAN_L: J3.2 (Pin_2), J4.2 (Pin_2), J5.2 (Pin_2), J6.2 (Pin_2), R2.2, R4.2, U1.6 (CANL)
- new net LED_1: R10.1, U4.27 (PB1)
- new net LED_2: R11.1, U4.28 (PB2)
- new net LED_3: R12.1, U4.57 (PB3(JTDO)
- new net LED_4: R13.1, U4.58 (PB4(NJTRST))
- new net LIMS1_1: D10.1 (K), J11.2 (Pin_2), R43.1, U4.24 (PC4)
- new net LIMS1_2: D16.1 (K), J12.2 (Pin_2), R51.1, U4.25 (PC5)
- new net LIMS2_1: D22.1 (K), J13.2 (Pin_2), R59.1, U4.40 (PC6)
- new net LIMS2_2: D25.1 (K), J14.2 (Pin_2), R65.1, U4.41 (PC7)
- new net LIMS3_1: D11.1 (K), J15.2 (Pin_2), R44.1, U4.42 (PC8)
- new net LIMS3_2: D17.1 (K), J16.2 (Pin_2), R52.1, U4.43 (PC9)
- new net LIMS4_1: D26.1 (K), J18.2 (Pin_2), R66.1, U4.55 (PC11)
- new net LIMS4_2: D23.1 (K), J17.2 (Pin_2), R60.1, U4.54 (PC10)
- new net NRST: C7.1, J19.1 (Pin_1), SW1.2, U4.7 (NRST)
- new net OSC: U17.3 (Output), U4.5 (PH0)
- new net POWER_MONITOR: U4.26 (PB0), U6.3
- new net Rol_SW1: SW3.1, U4.36 (PB14)
- new net Rol_SW2: SW3.2, U4.37 (PB15)
- new net Rol_SW4: SW3.4, U4.38 (PD11)
- new net Rol_SW8: SW3.8, U4.39 (PD12)
- new net SWCLK: J19.2 (Pin_2), U4.52 (PA14(JTCK)
- new net SWDIO: J19.3 (Pin_3), U4.49 (PA13(JTMS)
- new net Synchronization_Enable: R20.1, SW4.4
- new net Synchronization_Master: R19.1, SW4.3
- new net Synchronization_clock: J22.1 (Pin_1), R22.1, U4.16 (PA2)
- new net Synchronization_flag: J22.2 (Pin_2), R21.1, U4.20 (PA4)
- new net USB_DFU_DM: U18.A7 (D-), U18.B7 (D-), U4.47 (PA11)
- new net USB_DFU_DP: U18.A6 (D+), U18.B6 (D+), U4.48 (PA12)
- new net VBUS: C6.1, FB1.1, R23.1, U18.A4 (VBUS), U18.B4 (VBUS)
- new net VDD: C8.1, J20.1 (Pin_1), R14.1, R9.1, U5.4 (SHDN), U5.5 (Vin)
- new net XTAL_IN: C31.1, U4.3 (PC14), Y1.1 (X'tal)
- new net XTAL_OUT: C30.1, U4.4 (PC15), Y1.2 (X'tal)
- no-connect marks 0 -> 4
Other:
- note added: "FDCAN x1"
- note added: "HSE"
- note added: "LSE"
- note added: "NOR FLASH x1"
- note added: "STM-DFU"
- note added: "エンコーダー x4"
- note added: "リミットスイッチ x8"
- note added: "制御側電源"
- note added: "外部クロック"
- note added: "絶縁FDCAN x1"
- note added: "駆動側電源"
Changed lines of the file:
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@@
 	(generator "eeschema")
 	(generator_version "9.0")
-	(paper "A4")
-	(sheet_instances
-		(path "/"
-			(page "1")
-		)
-	)
-	(embedded_fonts no)
-)
+	(paper "A3")
