File: PCB/ESC_Device_Hub_v0/ESC_Device_Hub_v0.kicad_sch (KiCad schematic)
At the start: 137 parts, among them J1 Conn_01x04, J10 Conn_01x06, J11 Conn_01x02, J12 Conn_01x02, J13 Conn_01x02, J14 Conn_01x02, J15 Conn_01x02, J16 Conn_01x02, J17 Conn_01x02, J18 Conn_01x02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

Commit message: PCB完成
Other:
- note added: "FDCAN x2"
- note added: "絶縁FDCAN x4"
- note removed: "FDCAN x1"
- note removed: "絶縁FDCAN x1"
