File: PCB/ESC_Device_Hub_v0/ESC_Device_Hub_v0.kicad_pcb (KiCad board)
At the start: 2 copper layers, 50 x 90 mm, 141 parts, among them J1 Conn_01x04, J10 Conn_01x06, J11 Conn_01x02, J12 Conn_01x02, J13 Conn_01x02, J14 Conn_01x02, J15 Conn_01x02, J16 Conn_01x02, J17 Conn_01x02, J18 Conn_01x02, J19 Conn_01x05, J2 Conn_01x04, J20 Conn_01x01, J21 Conn_01x01, J22 Conn_01x02, J3 Conn_01x04, J4 Conn_01x04, J5 Conn_01x04, J6 Conn_01x04, J7 Conn_01x06, J8 Conn_01x06, J9 Conn_01x06, SW1 SW_Push, SW2 SW_Push, SW3 SW_Coded_SH-7050, SW4 SW_DIP_x02, U1 ISO1042BQDWVQ1, U18 USB_Type-C, U2 MCP2562FD-H/MF, U3 IS25LP064D-JLLE, U4 STM32H563RGVx, U5 NJW1933F1-AT, U6 TLP293, U7 NJM2884U1-33, U8 XC8114AA01PR-G, U9 XC8114AA01PR-G, Y1 FC2012SN 32.768K-70NNA0KC0

Commit message: PCB完成
Parts:
- moved J20 1.00 mm to (144.0, 101.0)
Routing:
- net GND: track 85.2 -> 165.6 mm, vias 21 -> 93
- net VBUS: track 14.2 -> 20.8 mm, vias 2 -> 3
- net USB_DFU_DP: track 9.06 -> 11.6 mm
- net USB_DFU_DM: track 9.10 -> 11.6 mm
- net ENC1_A: track 38.3 -> 40.0 mm
- net ENC1_B: track 44.8 -> 46.4 mm
- net +5V: track 158.5 -> 159.5 mm
- net FLASH_IO0: track 27.5 -> 28.3 mm
- net FLASH_SS: track 29.0 -> 29.7 mm
- net FLASH_IO1: track 27.5 -> 28.3 mm
- net FLASH_SCK: track 30.7 -> 31.5 mm
- net FLASH_IO3: track 27.6 -> 28.3 mm
- net FLASH_IO2: track 27.5 -> 28.3 mm
- net +5VA: track 40.7 -> 41.4 mm
- net POWER_MONITOR: track 68.9 -> 68.4 mm
Other:
- board text added: "+"
- board text added: "-"
- board text added: "120ohm"
