File: PCB/ESC_Device_Hub_v1/ESC_Device_Hub_v1.kicad_sch (KiCad schematic)
At the start: 131 parts, among them J1 Conn_01x04, J10 Conn_01x06, J11 Conn_01x02, J12 Conn_01x02, J13 Conn_01x02, J14 Conn_01x02, J15 Conn_01x02, J16 Conn_01x02, J17 Conn_01x02, J18 Conn_01x02, J19 Conn_01x05, J2 Conn_01x04, J20 Conn_01x01, J21 Conn_01x01, J22 Conn_01x02, J3 Conn_01x04, J4 Conn_01x04, J5 Conn_01x04, J6 Conn_01x04, J7 Conn_01x06, J8 Conn_01x06, J9 Conn_01x06, SW1 SW_Push, SW2 SW_Push, SW3 SW_Coded_SH-7050, U1 ISO1042BQDWVQ1, U10 LM66100DCK, U11 LM66100DCK, U18 USB_Type-C, U2 MCP2562FD-H/MF, U3 IS25LP064D-JLLE, U4 STM32H563RGVx, U6 TLP293, U7 NJM2884U1-33, U8 RFM-0505S, Y1 FC2012SN 32.768K-70NNA0KC0, Y2 XRCGB25M000FFS1AR0

Commit message: 残りLED
Parts:
- added R20, R6, R7: 1k, Resistor_SMD:R_0603_1608Metric_Pad0.98x0.95mm_HandSolder, symbol Device:R
Connections:
- net +3.3V: now also SW3.C; no longer R5.2
- net GND: now also R5.1, R20.1, R6.2, R7.2
- net LED_1: now also U4.15 (PA1)
- net LED_2: now also U4.14 (PA0)
- net LED_3: now also U4.11 (PC3)
- net LED_4: now also U4.10 (PC2)
- net Rol_SW1: now also R5.2
- net Rol_SW2: now also R6.1
- net Rol_SW4: now also U4.55 (PC11), R7.1; no longer U4.56 (PC12)
- net Rol_SW8: now also U4.56 (PC12), R20.2; no longer U4.55 (PC11)
- net Synchronization_clock: now also U4.17 (PA3)
- net Synchronization_flag: now also U4.16 (PA2)
- no-connect marks 7 -> 8
Other:
- moved on the sheet: SW3
