File: PCB/ESC_Device_Hub_v1/ESC_Device_Hub_v1.kicad_sch (KiCad schematic)
At the start: 130 parts, among them J1 Conn_01x04, J10 Conn_01x06, J11 Conn_01x02, J12 Conn_01x02, J13 Conn_01x02, J14 Conn_01x02, J15 Conn_01x02, J16 Conn_01x02, J17 Conn_01x02, J18 Conn_01x02, J19 Conn_01x05, J2 Conn_01x04, J20 Conn_01x01, J21 Conn_01x01, J22 Conn_01x02, J3 Conn_01x04, J4 Conn_01x04, J5 Conn_01x04, J6 Conn_01x04, J7 Conn_01x06, J8 Conn_01x06, J9 Conn_01x06, SW1 SW_Push, SW2 SW_Push, SW4 SW_DIP_x02, U1 ISO1042BQDWVQ1, U10 LM66100DCK, U11 LM66100DCK, U18 USB_Type-C, U2 MCP2562FD-H/MF, U3 IS25LP064D-JLLE, U4 STM32H563RGVx, U6 TLP293, U7 NJM2884U1-33, U8 RFM-0505S, Y1 FC2012SN 32.768K-70NNA0KC0, Y2 XRCGB25M000FFS1AR0

Commit message: PCBの更新
Connections:
- net +3.3V: now also J10.2 (Pin_2), J7.2 (Pin_2), J8.2 (Pin_2), J9.2 (Pin_2); no longer J10.5 (Pin_5), J7.5 (Pin_5), J8.5 (Pin_5), J9.5 (Pin_5)
- net ENC1_A: now also J8.1 (Pin_1); no longer J7.6 (Pin_6)
- net ENC1_B: now also J8.3 (Pin_3); no longer J7.4 (Pin_4)
- net ENC2_A: now also J7.1 (Pin_1); no longer J8.6 (Pin_6)
- net ENC2_B: now also J7.3 (Pin_3); no longer J8.4 (Pin_4)
- net ENC3_A: now also J10.1 (Pin_1); no longer J9.6 (Pin_6)
- net ENC3_B: now also J10.3 (Pin_3); no longer J9.4 (Pin_4)
- net ENC4_A: now also J9.1 (Pin_1); no longer J10.6 (Pin_6)
- net ENC4_B: now also J9.3 (Pin_3); no longer J10.4 (Pin_4)
- net GND: now also J10.4 (Pin_4), J10.5 (Pin_5), J10.6 (Pin_6), J19.3 (Pin_3), J7.4 (Pin_4), J7.5 (Pin_5), J7.6 (Pin_6), J8.4 (Pin_4), J8.5 (Pin_5), J8.6 (Pin_6), J9.4 (Pin_4), J9.5 (Pin_5), J9.6 (Pin_6); no longer J10.1 (Pin_1), J10.2 (Pin_2), J10.3 (Pin_3), J19.4 (Pin_4), J7.1 (Pin_1), J7.2 (Pin_2), J7.3 (Pin_3), J8.1 (Pin_1), J8.2 (Pin_2), J8.3 (Pin_3), J9.1 (Pin_1), J9.2 (Pin_2), J9.3 (Pin_3)
- net SWCLK: now also J19.4 (Pin_4); no longer J19.2 (Pin_2)
- net SWDIO: now also J19.2 (Pin_2); no longer J19.3 (Pin_3)
Other:
- moved on the sheet: J10, J7, J8, J9
