File: PCB/ESC_Device_Hub_v1/ESC_Device_Hub_v1.kicad_pcb (KiCad board)
At the start: 4 copper layers, 50 x 90 mm, 138 parts, among them J1 Conn_01x04, J10 Conn_01x06, J11 Conn_01x02, J12 Conn_01x02, J13 Conn_01x02, J14 Conn_01x02, J15 Conn_01x02, J16 Conn_01x02, J17 Conn_01x02, J18 Conn_01x02, J19 Conn_01x05, J2 Conn_01x04, J20 Conn_01x01, J21 Conn_01x01, J22 Conn_01x02, J3 Conn_01x04, J4 Conn_01x04, J5 Conn_01x04, J6 Conn_01x04, J7 Conn_01x06, J8 Conn_01x06, J9 Conn_01x06, SW1 SW_Push, SW2 SW_Push, SW3 SW_Coded_SH-7050, U1 ISO1042BQDWVQ1, U10 LM66100DCK, U11 LM66100DCK, U18 USB_Type-C, U2 MCP2562FD-H/MF, U3 IS25LP064D-JLLE, U4 STM32H563RGVx, U6 TLP293, U7 NJM2884U1-33, U8 RFM-0505S, Y1 FC2012SN 32.768K-70NNA0KC0, Y2 XRCGB25M000FFS1AR0

Commit message: 一部変更
Parts:
- removed R56: 1k, Resistor_SMD:R_0603_1608Metric_Pad0.98x0.95mm_HandSolder
- moved D1 18.0 mm to (150.4, 104.2)
- moved D2 18.0 mm to (150.4, 102.6)
- moved R14 18.0 mm to (153.7, 104.2)
- moved R8 18.0 mm to (153.7, 102.6)
- moved C31 0.47 mm to (158.6, 48.6)
- moved Y1 0.47 mm to (156.5, 49.1)
- moved C30 0.47 mm to (158.6, 49.5)
- moved C21 0.40 mm to (159.9, 47.6)
- moved C22 0.40 mm to (159.9, 46.7)
- moved C20 0.34 mm to (158.4, 46.5)
Connections:
- U6 pad 4: Net-(R56-Pad1) -> +3.3V
Routing:
- net +5VP: track 25.0 -> 43.1 mm
- net +5V: track 163.3 -> 149.5 mm
- net +3.3V: track 281.0 -> 276.2 mm, vias 13 -> 12
- net +5VA: track 103.3 -> 100.9 mm
- net ESC_FDCAN_TXD: track 44.2 -> 46.3 mm
- net Net-(R56-Pad1): track 1.79 -> 0.00 mm
- net VDD: track 39.0 -> 40.0 mm
- net ESC_FDCAN_RXD: track 43.1 -> 43.8 mm
- net GND: vias 74 -> 81
